File: garduino.sch (KiCad schematic (older format))
At the start: 14 parts, among them P1 GOOSVN, U1 CJT1117-5.0, U2 DS1339, U3 AT24CS16-STUM, Y1 32.768kHz

Commit message: Finished schematics
Parts:
- removed C1, C2, C3: 47u/25V, symbol CP
- removed C4, C6: C, symbol C
- removed FB1: FILTER, symbol FILTER
- removed U1: CJT1117-5.0, symbol AP1117D50
- added C1, C2: 10u/25V, Capacitors_SMD:C_0805, symbol C
- added C3, C5: 100n, Capacitors_SMD:C_0603, symbol C
- added P2: 3way KK, Connectors_Molex:Molex_KK_6410-03, symbol CONN_01X03
- added Q1: CJ2302, TO_SOT_Packages_SMD:SOT-23, symbol Q_NMOS_GSD
- added R2: 10k, Resistors_SMD:R_0603, symbol R
- C4: renamed from C5; footprint (none) -> jakub:SD_CAP; Manufacturer (none) -> Panasonic; Note (none) -> 330mF/5.5V ⌀10.5mm backup capacitor; Order Code (none) -> 2472068
- P1: value GOOSVN -> GS009S; footprint (none) -> Connect:AK300-2; Alt. Order Code (none) -> 320110028; Alt. Supplier (none) -> Open Parts Library; Manufacturer (none) -> GOOSVN; Note (none) -> 5mm 2way screw terminal; Order Code (none) -> 2493622; Package (none) -> 5mm pitch; Part Number (none) -> GS009S-5.0-02P-1; Supplier (none) -> Farnell
- R1: value 10k -> 560k; footprint (none) -> Resistors_SMD:R_0603; Alt. Order Code (none) -> 301010230; Alt. Supplier (none) -> Open Parts Library; Manufacturer (none) -> Yageo; Note (none) -> 560kΩ/5% 0603 resistor; Order Code (none) -> 9233717; Package (none) -> 0603; Part Number (none) -> RC0603JR-07560KL; Supplier (none) -> Farnell
- U1: renamed from U2; footprint (none) -> Housings_SSOP:MSOP-8_3x3mm_Pitch0.65mm; Manufacturer (none) -> Maxim; Note (none) -> I2C serial real-time clock; Order Code (none) -> 2515464; Package (none) -> USOP-8; Part Number (none) -> DS1339U-33+T&R; Supplier (none) -> Farnell
- U2: renamed from U3; value AT24CS16-STUM -> 24AA16T; footprint SOT-23-5 -> TO_SOT_Packages_SMD:SOT-23-5; Manufacturer (none) -> Microchip; Note (none) -> 16k I2C serial EEPROM; Order Code (none) -> 1331290; Package (none) -> SOT23-5; Part Number (none) -> 24AA16T-I/OT; Supplier (none) -> Farnell
- Y1: footprint (none) -> Crystals:Crystal_SMD_5032_2Pads; Alt. Order Code (none) -> 306010055; Alt. Supplier (none) -> Open Parts Library; Manufacturer (none) -> Xinhunjing; Note (none) -> 32768Hz 1206 7pF crystal; Order Code (none) -> 2467864; Package (none) -> 1206; Part Number (none) -> FC-135; Supplier (none) -> Farnell
Connections:
- net labels added: POWER, RELAY
- net labels removed: MOSI, Q0, Q1, Q2, Q3, Q4, Q5, Q6, Q7
- wire segments 79 -> 91
Other:
- moved on the sheet: A1, C4, U1, U2, Y1

Commit message: Laid out parts and routed some of the signals
Parts:
- A1: footprint (none) -> jakub:ARDUINO_MKR1000
Changed lines of the file:
@@
 F 0 "A1" H 2800 5800 60  0000 C CNN
 F 1 "ARDUINO_MKR1000" H 2800 3800 60  0000 C CNN
-F 2 "" H 2900 4550 60  0001 C CNN
+F 2 "jakub:ARDUINO_MKR1000" H 2900 4550 60  0001 C CNN
 F 3 "" H 2900 4550 60  0000 C CNN
 	1    2800 4550
