File: Sensors.sch (KiCad schematic (older format))
At the start: 18 parts, among them P10 CONN_01X03, P11 CONN_01X03, P12 CONN_01X03, P13 CONN_01X03, Q9 FDN340P, U5 MCP9700

Commit message: Finished schematics
Parts:
- removed P10, P11, P12, P13: CONN_01X03, symbol CONN_01X03
- removed R20: 150k, symbol R
- added C17, C20, C21, C22: 100n, Capacitors_SMD:C_0603, symbol C
- added P11, P12, P13, P14: 3pin 3.5mm jack, jakub:SUNTECH_ST-PJ-312, symbol ST-PJ-312
- added R23: 1k5, Resistors_SMD:R_0603, symbol R
- C15: renamed from C16; footprint (none) -> Capacitors_SMD:C_0603
- C16: renamed from C17; footprint (none) -> Capacitors_SMD:C_0603
- C18, C19: footprint (none) -> Capacitors_SMD:C_0603
- C23: renamed from C?; footprint (none) -> Capacitors_SMD:C_0603
- D17: footprint (none) -> Diodes_SMD:SMA_Standard
- Q10: renamed from Q9; footprint (none) -> TO_SOT_Packages_SMD:SOT-23
- R19: renamed from R18; footprint (none) -> Resistors_SMD:R_0603
- R20: renamed from R19; footprint (none) -> Resistors_SMD:R_0603
- R21: value 1k5 -> 560k; footprint (none) -> Resistors_SMD:R_0603; Alt. Order Code 301010114 -> 301010230; Note 1.5kΩ/1% 0603 resistor -> 560kΩ/5% 0603 resistor; Order Code 9233407 -> 9233717; Part Number RC0603JR-071K5L -> RC0603JR-07560KL
- R22: footprint (none) -> Resistors_SMD:R_0603
- R24: renamed from R23; footprint (none) -> Resistors_SMD:R_0603
- U4: renamed from U5; footprint (none) -> TO_SOT_Packages_SMD:SOT-23
Connections:
- net +3V3: now also R21.1
- net GND: now also C17.2, C20.2, C21.2, C22.2, P11.COM1, P11.COM2, P12.COM1, P12.COM2, P13.COM1, P13.COM2, P14.COM1, P14.COM2
- net SENS2: now also R22.2; no longer R21.2
- net SENS3: now also R23.2; no longer R22.2
- net at C15.1, R19.1: now also P11.R
- net at Q10.3 (D): now also C18.1, C17.1, C21.1, C22.1, P11.L, P12.L, P13.L, P14.L
- net at C16.1, R20.1: now also P12.R
- net at C19.1, R22.1: now also P13.R
- net at D17.2 (A), Q10.1 (G): now also R21.2
- new net: C20.1, P14.R, R23.1
- no-connect marks 0 -> 8
Other:
- moved on the sheet: C15, C16, C23, D17, Q10, R19, R20, R24, U4

Commit message: Final production board
Other:
- note added: "FOUR EXTERANAL SENSOR CONNECTORS"
- note added: "SENSOR POWER SWITCH"
- note added: "SENSORS\nUp to four external sensors powered by 3.3V can be connected through 3.5mm audio jacks.\nThe power supply to the sensors is controlled by the Arduino to conserve power and minimize electrolytic damage to moisture sensors.\nThe idea is to probe the sensors only at pre-programmed intervals.\nThere is a temperature sensor on board to allow following the temperature. This might be particular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"
- note added: "TEMPERATURE SENSOR"
Changed lines of the file:
@@
 LIBS:valves
 LIBS:jakub
-LIBS:garduino-cache
+LIBS:guarduino-cache
 EELAYER 25 0
 EELAYER END
@@
 encoding utf-8
 Sheet 3 4
-Title ""
-Date ""
-Rev ""
-Comp ""
-Comment1 ""
-Comment2 ""
+Title "Guarduino Control Unit"
+Date "2016-09-30"
+Rev "1.0"
+Comp "Serious Play Ltd"
+Comment1 "Jakub Nedbal"
+Comment2 "License: CC-BY-SA"
 Comment3 ""
 Comment4 ""
@@
 U 1 1 576A862F
 P 3000 3550
-F 0 "P11" H 2800 3600 50  0000 L BNN
-F 1 "3pin 3.5mm jack" H 2800 3500 50  0000 L TNN
+F 0 "P11" H 2750 3600 50  0000 L BNN
+F 1 "3pin 3.5mm jack" H 2750 3500 50  0000 L TNN
 F 2 "jakub:SUNTECH_ST-PJ-312" H 3000 3550 50  0001 L CNN
 F 3 "" H 3000 3550 60  0000 C CNN
@@
 U 1 1 576AA5E8
 P 3000 5450
-F 0 "P12" H 2800 5500 50  0000 L BNN
-F 1 "3pin 3.5mm jack" H 2800 5400 50  0000 L TNN
+F 0 "P12" H 2750 5500 50  0000 L BNN
+F 1 "3pin 3.5mm jack" H 2750 5400 50  0000 L TNN
 F 2 "jakub:SUNTECH_ST-PJ-312" H 3000 5450 50  0001 L CNN
 F 3 "" H 3000 5450 60  0000 C CNN
@@
 U 1 1 576AA684
 P 7000 5450
-F 0 "P14" H 6800 5500 50  0000 L BNN
-F 1 "3pin 3.5mm jack" H 6800 5400 50  0000 L TNN
+F 0 "P14" H 6750 5500 50  0000 L BNN
+F 1 "3pin 3.5mm jack" H 6750 5400 50  0000 L TNN
 F 2 "jakub:SUNTECH_ST-PJ-312" H 7000 5450 50  0001 L CNN
 F 3 "" H 7000 5450 60  0000 C CNN
@@
 U 1 1 576AA729
 P 7000 3550
-F 0 "P13" H 6800 3600 50  0000 L BNN
-F 1 "3pin 3.5mm jack" H 6800 3500 50  0000 L TNN
+F 0 "P13" H 6750 3600 50  0000 L BNN
+F 1 "3pin 3.5mm jack" H 6750 3500 50  0000 L TNN
 F 2 "jakub:SUNTECH_ST-PJ-312" H 7000 3550 50  0001 L CNN
 F 3 "" H 7000 3550 60  0000 C CNN
@@
 Connection ~ 7700 5700
 Connection ~ 3700 5700
+Text Notes 750  1300 0    60   ~ 0
+SENSORS\nUp to four external sensors powered by 3.3V can be connected through 3.5mm audio jacks.\nThe power supply to the sensors is controlled by the Arduino to conserve power and minimize electrolytic damage to moisture sensors.\nThe idea is to probe the sensors only at pre-programmed intervals.\nThere is a temperature sensor on board to allow following the temperature. This might be particularly useful to turn-off watering or draining the pipes during frosts.
+Text Notes 3200 1550 0    60   ~ 0
+SENSOR POWER SWITCH
+Text Notes 4050 2100 0    60   ~ 0
+FOUR EXTERANAL SENSOR CONNECTORS
+Text Notes 8700 2100 0    60   ~ 0
+TEMPERATURE SENSOR
 $EndSCHEMATC
