File: RFmodules.sch (KiCad schematic (older format))
At the start: 14 parts, among them M1 PT2272, M2 PT2272, U6 74AHC1G02, U7 74HCT165, U8 74AHCT1G125

Commit message: Finished schematics
Parts:
- C24: renamed from C21; footprint (none) -> Capacitors_SMD:C_0603
- C25: renamed from C22; footprint (none) -> Capacitors_SMD:C_0603
- C26: renamed from C23; footprint (none) -> Capacitors_SMD:C_0603
- C27: renamed from C24; footprint (none) -> Capacitors_SMD:C_0603
- C28: renamed from C25; footprint (none) -> Capacitors_SMD:C_0603
- M1, M2: footprint (none) -> Socket_Strips:Socket_Strip_Straight_1x07
- R25: renamed from R24; footprint (none) -> Resistors_SMD:R_0603
- R26: renamed from R25; footprint (none) -> Resistors_SMD:R_0603
- R27: renamed from R26; footprint (none) -> Resistors_SMD:R_0603
- R28: renamed from R27; footprint (none) -> Resistors_SMD:R_0603
- U5: renamed from U6; footprint (none) -> TO_SOT_Packages_SMD:SC-70-5
- U6: renamed from U7; footprint (none) -> Housings_SOIC:SOIC-16_3.9x9.9mm_Pitch1.27mm
- U7: renamed from U8; footprint (none) -> TO_SOT_Packages_SMD:SC-70-5
Changed lines of the file:
@@
 $EndDescr
 $Comp
-L 74LS165 U7
+L 74LS165 U6
 U 1 1 570BE18F
 P 4800 4400
-F 0 "U7" H 4800 5100 50  0000 C CNN
+F 0 "U6" H 4800 5100 50  0000 C CNN
 F 1 "74HCT165" H 4800 3700 50  0000 C CNN
-F 2 "" H 4800 4400 50  0000 C CNN
+F 2 "Housings_SOIC:SOIC-16_3.9x9.9mm_Pitch1.27mm" H 4800 4400 50  0001 C CNN
 F 3 "" H 4800 4400 50  0000 C CNN
 F 4 "CD74HCT165M96" H 4800 4400 60  0001 C CNN "Part Number"
@@
 $EndComp
 $Comp
-L 74HCT1G125 U8
+L 74HCT1G125 U7
 U 1 1 570BE197
 P 6400 3900
-F 0 "U8" H 6400 4100 60  0000 C CNN
+F 0 "U7" H 6400 4100 60  0000 C CNN
 F 1 "74AHCT1G125" H 6400 3550 60  0000 C CNN
-F 2 "" H 6400 3900 60  0000 C CNN
+F 2 "TO_SOT_Packages_SMD:SC-70-5" H 6400 3900 60  0001 C CNN
 F 3 "" H 6400 3900 60  0000 C CNN
 F 4 "SN74AHCT1G125DCKT" H 6400 3900 60  0001 C CNN "Part Number"
@@
 $EndComp
 $Comp
-L GND #PWR92
+L GND #PWR093
 U 1 1 570BE1AC
 P 7400 4500
-F 0 "#PWR92" H 7400 4250 50  0001 C CNN
+F 0 "#PWR093" H 7400 4250 50  0001 C CNN
 F 1 "GND" H 7400 4350 50  0000 C CNN
 F 2 "" H 7400 4500 50  0000 C CNN
@@
 F 0 "M1" H 100 1600 60  0000 L CNN
 F 1 "PT2272" H 100 1500 60  0000 L CNN
-F 2 "" H 1700 1400 60  0000 C CNN
+F 2 "Socket_Strips:Socket_Strip_Straight_1x07" H 1700 1400 60  0001 C CNN
 F 3 "" H 1700 1400 60  0000 C CNN
 	1    1700 1400
@@
 F 0 "M2" H 2300 1600 60  0000 L CNN
 F 1 "PT2272" H 2300 1500 60  0000 L CNN
-F 2 "" H 3900 1400 60  0000 C CNN
+F 2 "Socket_Strips:Socket_Strip_Straight_1x07" H 3900 1400 60  0001 C CNN
 F 3 "" H 3900 1400 60  0000 C CNN
 	1    3900 1400
@@
 VT_1
 $Comp
-L GND #PWR81
+L GND #PWR094
 U 1 1 570BE1D9
 P 2000 2100
-F 0 "#PWR81" H 2000 1850 50  0001 C CNN
+F 0 "#PWR094" H 2000 1850 50  0001 C CNN
 F 1 "GND" H 2000 1950 50  0000 C CNN
 F 2 "" H 2000 2100 50  0000 C CNN
@@
 $EndComp
 $Comp
-L VCC #PWR82
+L VCC #PWR095
 U 1 1 570BE1DF
 P 2100 1300
-F 0 "#PWR82" H 2100 1150 50  0001 C CNN
+F 0 "#PWR095" H 2100 1150 50  0001 C CNN
 F 1 "VCC" H 2100 1450 50  0000 C CNN
 F 2 "" H 2100 1300 50  0000 C CNN
@@
 VT_2
 $Comp
-L GND #PWR86
+L GND #PWR096
 U 1 1 570BE1EA
 P 4200 2100
-F 0 "#PWR86" H 4200 1850 50  0001 C CNN
+F 0 "#PWR096" H 4200 1850 50  0001 C CNN
 F 1 "GND" H 4200 1950 50  0000 C CNN
 F 2 "" H 4200 2100 50  0000 C CNN
@@
 $EndComp
 $Comp
-L VCC #PWR87
+L VCC #PWR097
 U 1 1 570BE1F0
 P 4300 1300
-F 0 "#PWR87" H 4300 1150 50  0001 C CNN
+F 0 "#PWR097" H 4300 1150 50  0001 C CNN
 F 1 "VCC" H 4300 1450 50  0000 C CNN
 F 2 "" H 4300 1300 50  0000 C CNN
@@
 	4200 1400 4200 2100
 $Comp
-L 74AHC1G02 U6
+L 74AHC1G02 U5
 U 1 1 570BE4CA
 P 2500 4750
-F 0 "U6" H 2500 4800 50  0000 C CNN
+F 0 "U5" H 2500 4800 50  0000 C CNN
 F 1 "74AHC1G02" H 2550 4700 50  0000 C CNN
-F 2 "" H 2500 4750 50  0000 C CNN
+F 2 "TO_SOT_Packages_SMD:SC-70-5" H 2500 4750 50  0001 C CNN
 F 3 "" H 2500 4750 50  0000 C CNN
 F 4 "SN74AHC1G02DCKR" H 2500 4750 60  0001 C CNN "Part Number"
@@
 MISO
 $Comp
-L R R24
+L R R25
 U 1 1 570BEB97
 P 3550 5600
-F 0 "R24" V 3630 5600 50  0000 C CNN
+F 0 "R25" V 3630 5600 50  0000 C CNN
 F 1 "1k5" V 3550 5600 50  0000 C CNN
-F 2 "" V 3480 5600 50  0000 C CNN
+F 2 "Resistors_SMD:R_0603" V 3480 5600 50  0001 C CNN
 F 3 "" H 3550 5600 50  0000 C CNN
 F 4 "RC0603JR-071K5L" H 3550 5600 60  0001 C CNN "Part Number"
@@
 $EndComp
 $Comp
-L R R25
+L R R26
 U 1 1 570BEB9D
 P 3800 5850
-F 0 "R25" V 3880 5850 50  0000 C CNN
+F 0 "R26" V 3880 5850 50  0000 C CNN
 F 1 "3k" V 3800 5850 50  0000 C CNN
-F 2 "" V 3730 5850 50  0000 C CNN
+F 2 "Resistors_SMD:R_0603" V 3730 5850 50  0001 C CNN
 F 3 "" H 3800 5850 50  0000 C CNN
 F 4 "RC0603FR-073KL" H 3800 5850 60  0001 C CNN "Part Number"
@@
 $EndComp
 $Comp
-L GND #PWR85
+L GND #PWR098
 U 1 1 570BEBA3
 P 3800 6200
-F 0 "#PWR85" H 3800 5950 50  0001 C CNN
+F 0 "#PWR098" H 3800 5950 50  0001 C CNN
 F 1 "GND" H 3800 6050 50  0000 C CNN
 F 2 "" H 3800 6200 50  0000 C CNN
@@
 $EndComp
 $Comp
-L C C22
+L C C25
 U 1 1 570BEBA9
 P 3550 5400
-F 0 "C22" V 3400 5450 50  0000 L CNN
+F 0 "C25" V 3400 5450 50  0000 L CNN
 F 1 "10p" V 3500 5450 50  0000 L CNN
-F 2 "" H 3588 5250 50  0000 C CNN
+F 2 "Capacitors_SMD:C_0603" H 3588 5250 50  0001 C CNN
 F 3 "" H 3550 5400 50  0000 C CNN
 F 4 "CC0603JRNPO9BN100" H 3550 5400 60  0001 C CNN "Part Number"
@@
 SD2
 $Comp
-L C C21
+L C C24
 U 1 1 570C68DF
 P 2500 5950
-F 0 "C21" H 2525 6050 50  0000 L CNN
+F 0 "C24" H 2525 6050 50  0000 L CNN
 F 1 "100n" H 2525 5850 50  0000 L CNN
-F 2 "" H 2538 5800 50  0000 C CNN
+F 2 "Capacitors_SMD:C_0603" H 2538 5800 50  0001 C CNN
 F 3 "" H 2500 5950 50  0000 C CNN
 F 4 "CC0603KRX7R9BB104" H 2500 5950 60  0001 C CNN "Part Number"
@@
 	2500 6100 2500 6200
 $Comp
-L GND #PWR84
+L GND #PWR099
 U 1 1 570C68E7
 P 2500 6200
-F 0 "#PWR84" H 2500 5950 50  0001 C CNN
+F 0 "#PWR099" H 2500 5950 50  0001 C CNN
 F 1 "GND" H 2500 6050 50  0000 C CNN
 F 2 "" H 2500 6200 50  0000 C CNN
@@
 	2500 5800 2500 5700
 $Comp
-L VCC #PWR83
+L VCC #PWR0100
 U 1 1 570C68EE
 P 2500 5700
-F 0 "#PWR83" H 2500 5550 50  0001 C CNN
+F 0 "#PWR0100" H 2500 5550 50  0001 C CNN
 F 1 "VCC" H 2500 5850 50  0000 C CNN
 F 2 "" H 2500 5700 50  0000 C CNN
@@
 	5500 5200 5500 5300
 $Comp
-L GND #PWR89
+L GND #PWR0101
 U 1 1 570C6A23
 P 5500 5300
-F 0 "#PWR89" H 5500 5050 50  0001 C CNN
+F 0 "#PWR0101" H 5500 5050 50  0001 C CNN
 F 1 "GND" H 5500 5150 50  0000 C CNN
 F 2 "" H 5500 5300 50  0000 C CNN
@@
 	5500 4900 5500 4800
 $Comp
-L VCC #PWR88
+L VCC #PWR0102
 U 1 1 570C6A2A
 P 5500 4800
-F 0 "#PWR88" H 5500 4650 50  0001 C CNN
+F 0 "#PWR0102" H 5500 4650 50  0001 C CNN
 F 1 "VCC" H 5500 4950 50  0000 C CNN
 F 2 "" H 5500 4800 50  0000 C CNN
@@
 	6400 5200 6400 5300
 $Comp
-L GND #PWR91
+L GND #PWR0103
 U 1 1 570C6B23
 P 6400 5300
-F 0 "#PWR91" H 6400 5050 50  0001 C CNN
+F 0 "#PWR0103" H 6400 5050 50  0001 C CNN
 F 1 "GND" H 6400 5150 50  0000 C CNN
 F 2 "" H 6400 5300 50  0000 C CNN
@@
 	6400 4900 6400 4800
 $Comp
-L VCC #PWR90
+L VCC #PWR0104
 U 1 1 570C6B2A
 P 6400 4800
-F 0 "#PWR90" H 6400 4650 50  0001 C CNN
+F 0 "#PWR0104" H 6400 4650 50  0001 C CNN
 F 1 "VCC" H 6400 4950 50  0000 C CNN
 F 2 "" H 6400 4800 50  0000 C CNN
@@
 $EndComp
 $Comp
-L C C23
+L C C26
 U 1 1 573D12B0
 P 5500 5050
-F 0 "C23" H 5525 5150 50  0000 L CNN
+F 0 "C26" H 5525 5150 50  0000 L CNN
 F 1 "100n" H 5525 4950 50  0000 L CNN
-F 2 "" H 5538 4900 50  0000 C CNN
+F 2 "Capacitors_SMD:C_0603" H 5538 4900 50  0001 C CNN
 F 3 "" H 5500 5050 50  0000 C CNN
 F 4 "CC0603KRX7R9BB104" H 5500 5050 60  0001 C CNN "Part Number"
@@
 $EndComp
 $Comp
-L C C24
+L C C27
 U 1 1 573D1332
 P 6400 5050
-F 0 "C24" H 6425 5150 50  0000 L CNN
+F 0 "C27" H 6425 5150 50  0000 L CNN
 F 1 "100n" H 6425 4950 50  0000 L CNN
-F 2 "" H 6438 4900 50  0000 C CNN
+F 2 "Capacitors_SMD:C_0603" H 6438 4900 50  0001 C CNN
 F 3 "" H 6400 5050 50  0000 C CNN
 F 4 "CC0603KRX7R9BB104" H 6400 5050 60  0001 C CNN "Part Number"
@@
 $EndComp
 $Comp
-L C C25
+L C C28
 U 1 1 573D1776
 P 7150 3700
-F 0 "C25" V 7000 3750 50  0000 L CNN
+F 0 "C28" V 7000 3750 50  0000 L CNN
 F 1 "10p" V 7100 3750 50  0000 L CNN
-F 2 "" H 7188 3550 50  0000 C CNN
+F 2 "Capacitors_SMD:C_0603" H 7188 3550 50  0001 C CNN
 F 3 "" H 7150 3700 50  0000 C CNN
 F 4 "CC0603JRNPO9BN100" H 7150 3700 60  0001 C CNN "Part Number"
@@
 $EndComp
 $Comp
-L R R26
+L R R27
 U 1 1 573D3924
 P 7150 3900
-F 0 "R26" V 7230 3900 50  0000 C CNN
+F 0 "R27" V 7230 3900 50  0000 C CNN
 F 1 "1k5" V 7150 3900 50  0000 C CNN
-F 2 "" V 7080 3900 50  0000 C CNN
+F 2 "Resistors_SMD:R_0603" V 7080 3900 50  0001 C CNN
 F 3 "" H 7150 3900 50  0000 C CNN
 F 4 "RC0603JR-071K5L" H 7150 3900 60  0001 C CNN "Part Number"
@@
 $EndComp
 $Comp
-L R R27
+L R R28
 U 1 1 573D3D7C
 P 7400 4150
-F 0 "R27" V 7480 4150 50  0000 C CNN
+F 0 "R28" V 7480 4150 50  0000 C CNN
 F 1 "3k" V 7400 4150 50  0000 C CNN
-F 2 "" V 7330 4150 50  0000 C CNN
+F 2 "Resistors_SMD:R_0603" V 7330 4150 50  0001 C CNN
 F 3 "" H 7400 4150 50  0000 C CNN
 F 4 "RC0603FR-073KL" H 7400 4150 60  0001 C CNN "Part Number"

Commit message: Final production board
Other:
- note added: "3-STATE DRIVER"
- note added: "DATA LATCH\nStore current state of outputs of both\nRF modules in the input latch of the\nserial-to-parallel shift register."
- note added: "INTERRUPT OUTPUT\ncalled when RF data is received"
- note added: "PARALLEL-TO-SERIAL SHIFT REGISTER"
- note added: "RF MODULES\nTwo wireless 433MHz modules with four channels each can be used to provide input to the control unit.\nWhenever any of the RF modules receives an input, it signals to the Arduino, which consequently reads out which channel was called.\nThere is a parallel-to-serial shift register to allow readout of the eight inputs.\nAs the RF modules use 5V power supply, their outputs are divided by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"
- note added: "TWO 433 MHz RF MODULES"
- moved on the sheet: C24, C25, C26, C27, C28, M1, M2, R25, R26, R27, R28, U5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

Commit message: Fixed order codes
Parts:
- C24, C26, C27: Alt. Order Code (none) -> 302010138
- C25, C28: Alt. Order Code (none) -> 302010097
- R26, R28: Alt. Order Code (none) -> 301010170
Changed lines of the file:
@@
 F 8 "9330976" H 3800 6250 60  0001 C CNN "Order Code"
 F 9 "Open Parts Library" H 3800 6250 60  0001 C CNN "Alt. Supplier"
-F 10 "3kΩ/1% 0603 resistor" H 3800 6250 60  0001 C CNN "Note"
+F 10 "301010170" H 3800 6250 60  0001 C CNN "Alt. Order Code"
+F 11 "3kΩ/1% 0603 resistor" H 3800 6250 60  0001 C CNN "Note"
 	1    3800 6250
 	1    0    0    -1
@@
 F 8 "721967" H 3550 5800 60  0001 C CNN "Order Code"
 F 9 "Open Parts Library" H 3550 5800 60  0001 C CNN "Alt. Supplier"
-F 10 "10pF/50V C0G/NP0 0603 ceramic capacitor" H 3550 5800 60  0001 C CNN "Note"
+F 10 "302010097" H 3550 5800 60  0001 C CNN "Alt. Order Code"
+F 11 "10pF/50V C0G/NP0 0603 ceramic capacitor" H 3550 5800 60  0001 C CNN "Note"
 	1    3550 5800
 	0    1    1    0
@@
 F 8 "1362556" H 2500 6350 60  0001 C CNN "Order Code"
 F 9 "Open Parts Library" H 2500 6350 60  0001 C CNN "Alt. Supplier"
-F 10 "100nF/50V X7R 0603 ceramic capacitor" H 2500 6350 60  0001 C CNN "Note"
+F 10 "302010138" H 2500 6350 60  0001 C CNN "Alt. Order Code"
+F 11 "100nF/50V X7R 0603 ceramic capacitor" H 2500 6350 60  0001 C CNN "Note"
 	1    2500 6350
 	1    0    0    -1
@@
 F 8 "1362556" H 5500 5450 60  0001 C CNN "Order Code"
 F 9 "Open Parts Library" H 5500 5450 60  0001 C CNN "Alt. Supplier"
-F 10 "100nF/50V X7R 0603 ceramic capacitor" H 5500 5450 60  0001 C CNN "Note"
+F 10 "302010138" H 5500 5450 60  0001 C CNN "Alt. Order Code"
+F 11 "100nF/50V X7R 0603 ceramic capacitor" H 5500 5450 60  0001 C CNN "Note"
 	1    5500 5450
 	1    0    0    -1
@@
 F 8 "1362556" H 6400 5450 60  0001 C CNN "Order Code"
 F 9 "Open Parts Library" H 6400 5450 60  0001 C CNN "Alt. Supplier"
-F 10 "100nF/50V X7R 0603 ceramic capacitor" H 6400 5450 60  0001 C CNN "Note"
+F 10 "302010138" H 6400 5450 60  0001 C CNN "Alt. Order Code"
+F 11 "100nF/50V X7R 0603 ceramic capacitor" H 6400 5450 60  0001 C CNN "Note"
 	1    6400 5450
 	1    0    0    -1
@@
 F 8 "721967" H 7150 4100 60  0001 C CNN "Order Code"
 F 9 "Open Parts Library" H 7150 4100 60  0001 C CNN "Alt. Supplier"
-F 10 "10pF/50V C0G/NP0 0603 ceramic capacitor" H 7150 4100 60  0001 C CNN "Note"
+F 10 "302010097" H 7150 4100 60  0001 C CNN "Alt. Order Code"
+F 11 "10pF/50V C0G/NP0 0603 ceramic capacitor" H 7150 4100 60  0001 C CNN "Note"
 	1    7150 4100
 	0    1    1    0
@@
 F 8 "9330976" H 7400 4550 60  0001 C CNN "Order Code"
 F 9 "Open Parts Library" H 7400 4550 60  0001 C CNN "Alt. Supplier"
-F 10 "3kΩ/1% 0603 resistor" H 7400 4550 60  0001 C CNN "Note"
+F 10 "301010170" H 7400 4550 60  0001 C CNN "Alt. Order Code"
+F 11 "3kΩ/1% 0603 resistor" H 7400 4550 60  0001 C CNN "Note"
 	1    7400 4550
 	1    0    0    -1
