File: guarduino.sch (KiCad schematic (older format))
At the start: 14 parts, among them P1 GS009S, P2 3way KK, Q1 CJ2302, U1 DS1339, U2 24AA16T, Y1 32.768kHz

Commit message: Final production board
Parts:
- removed P1: GS009S, Connect:AK300-2, symbol CONN_01X02
- removed P2: 3way KK, Connectors_Molex:Molex_KK_6410-03, symbol CONN_01X03
- added H1, H2, H3, H4: ⌀3mm, Mounting_Holes:MountingHole_3.2mm_M3, symbol CONN_01X01
- added P1: 4way mini DIN, jakub:MiniDIN4way, symbol CONN_01X05
- added P2: 4way connector, jakub:JST_PH_04way_vert, symbol CONN_01X04
Connections:
- wire segments 91 -> 94
- no-connect marks 3 -> 8
Other:
- note added: "EEPROM"
- note added: "GROVE CONNECTOR\nConnect to Raining Cats\npower supply using 5cm\ngrove cable\nSKU: 110990036"
- note added: "HIGH CURRENT POWER SUPPLY SWITCH"
- note added: "MOUNTING HOLES"
- note added: "REAL TIME CLOCK"
- moved on the sheet: C1, C2, Q1, R1

Commit message: Fixed order codes
Parts:
- C3, C5: Alt. Order Code (none) -> 302010138
Changed lines of the file:
@@
 F 8 "1362556" H 6700 3450 60  0001 C CNN "Order Code"
 F 9 "Open Parts Library" H 6700 3450 60  0001 C CNN "Alt. Supplier"
-F 10 "100nF/50V X7R 0603 ceramic capacitor" H 6700 3450 60  0001 C CNN "Note"
+F 10 "302010138" H 6700 3450 60  0001 C CNN "Alt. Order Code"
+F 11 "100nF/50V X7R 0603 ceramic capacitor" H 6700 3450 60  0001 C CNN "Note"
 	1    6700 3450
 	1    0    0    -1
@@
 F 8 "1362556" H 9300 3450 60  0001 C CNN "Order Code"
 F 9 "Open Parts Library" H 9300 3450 60  0001 C CNN "Alt. Supplier"
-F 10 "100nF/50V X7R 0603 ceramic capacitor" H 9300 3450 60  0001 C CNN "Note"
+F 10 "302010138" H 9300 3450 60  0001 C CNN "Alt. Order Code"
+F 11 "100nF/50V X7R 0603 ceramic capacitor" H 9300 3450 60  0001 C CNN "Note"
 	1    9300 3450
 	1    0    0    -1
